File: code arduino et fichiers kicad/kicad/pcb.kicad_sch (KiCad schematic)
At the start: 46 parts, among them J1 Screw_Terminal_01x04, J2 Screw_Terminal_01x02, U1 LMC6482, U2 LMC6482, U3 LMC6482, U4 LMC6482

Commit message: PC V2 fini
Parts:
- U1, U2, U3, U4: footprint ampli op:LMC6482 -> ampli op:LMC6482_SMT
Connections:
- net +5V: no longer J1.4 (Pin_4), J2.2 (Pin_2)
- net T1 sortie: now also analogA0-A7.4 (Pin_4); no longer analogA0-A7.1 (Pin_1)
- net T2 sortie: now also analogA0-A7.3 (Pin_3); no longer analogA0-A7.2 (Pin_2)
- net T3 sortie: now also analogA0-A7.2 (Pin_2); no longer analogA0-A7.3 (Pin_3)
- net T4 sortie: now also analogA0-A7.1 (Pin_1); no longer analogA0-A7.4 (Pin_4)
- net pwmdroite: now also J1.1 (Pin_1); no longer J1.2 (Pin_2)
- net pwmgauche: now also J1.2 (Pin_2); no longer J1.1 (Pin_1)
- new net +5V (Ali seulement): J1.4 (Pin_4), J2.2 (Pin_2)
Changed lines of the file:
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@@
 	(wire
 		(pts
-			(xy 218.44 83.82) (xy 218.44 91.44)
-		)
-		(stroke
-			(width 0)
-			(type default)
-		)
-	)
-	(wire
-		(pts
 			(xy 83.82 27.94) (xy 93.98 27.94)
 		)
@@
 	(wire
 		(pts
-			(xy 215.9 78.74) (xy 231.14 78.74)
-		)
-		(stroke
-			(width 0)
-			(type default)
-		)
-	)
-	(wire
-		(pts
 			(xy 78.74 101.6) (xy 76.2 101.6)
 		)
@@
 	(wire
 		(pts
-			(xy 33.02 143.51) (xy 41.91 143.51)
-		)
-		(stroke
-			(width 0)
-			(type default)
-		)
-	)
-	(wire
-		(pts
 			(xy 252.73 55.88) (xy 261.62 55.88)
 		)
@@
 	(wire
 		(pts
+			(xy 220.98 91.44) (xy 215.9 91.44)
+		)
+		(stroke
+			(width 0)
+			(type default)
+		)
+	)
+	(wire
+		(pts
 			(xy 123.19 41.91) (xy 127 41.91)
 		)
@@
 	(wire
 		(pts
-			(xy 218.44 83.82) (xy 231.14 83.82)
-		)
-		(stroke
-			(width 0)
-			(type default)
-		)
-	)
-	(wire
-		(pts
 			(xy 231.14 57.15) (xy 213.36 57.15)
 		)
@@
 	(wire
 		(pts
-			(xy 215.9 97.79) (xy 220.98 97.79)
+			(xy 213.36 57.15) (xy 213.36 44.45)
 		)
 		(stroke
@@
 	(wire
 		(pts
-			(xy 213.36 57.15) (xy 213.36 44.45)
+			(xy 121.92 78.74) (xy 144.78 78.74)
 		)
 		(stroke
@@
 	(wire
 		(pts
-			(xy 121.92 78.74) (xy 144.78 78.74)
+			(xy 215.9 81.28) (xy 231.14 81.28)
 		)
 		(stroke
@@
 	(wire
 		(pts
+			(xy 222.25 78.74) (xy 231.14 78.74)
+		)
+		(stroke
+			(width 0)
+			(type default)
+		)
+	)
+	(wire
+		(pts
 			(xy 139.7 104.14) (xy 142.24 104.14)
 		)
@@
 	(wire
 		(pts
+			(xy 218.44 86.36) (xy 218.44 83.82)
+		)
+		(stroke
+			(width 0)
+			(type default)
+		)
+	)
+	(wire
+		(pts
 			(xy 231.14 62.23) (xy 228.6 62.23)
 		)
@@
 	(wire
 		(pts
-			(xy 220.98 97.79) (xy 220.98 86.36)
-		)
-		(stroke
-			(width 0)
-			(type default)
-		)
-	)
-	(wire
-		(pts
 			(xy 74.93 86.36) (xy 80.01 86.36)
 		)
@@
 	(wire
 		(pts
+			(xy 215.9 76.2) (xy 222.25 76.2)
+		)
+		(stroke
+			(width 0)
+			(type default)
+		)
+	)
+	(wire
+		(pts
 			(xy 175.26 30.48) (xy 170.18 30.48)
 		)
@@
 	(wire
 		(pts
-			(xy 217.17 81.28) (xy 231.14 81.28)
-		)
-		(stroke
-			(width 0)
-			(type default)
-		)
-	)
-	(wire
-		(pts
-			(xy 215.9 91.44) (xy 218.44 91.44)
-		)
-		(stroke
-			(width 0)
-			(type default)
-		)
-	)
-	(wire
-		(pts
 			(xy 93.98 81.28) (xy 93.98 91.44)
 		)
@@
 	(wire
 		(pts
-			(xy 215.9 85.09) (xy 217.17 85.09)
-		)
-		(stroke
-			(width 0)
-			(type default)
-		)
-	)
-	(wire
-		(pts
 			(xy 157.48 22.86) (xy 157.48 30.48)
 		)
@@
 	(wire
 		(pts
+			(xy 30.48 143.51) (xy 41.91 143.51)
+		)
+		(stroke
+			(width 0)
+			(type default)
+		)
+	)
+	(wire
+		(pts
 			(xy 157.48 30.48) (xy 162.56 30.48)
 		)
@@
 	(wire
 		(pts
-			(xy 217.17 85.09) (xy 217.17 81.28)
+			(xy 40.64 53.34) (xy 40.64 54.61)
 		)
 		(stroke
@@
 	(wire
 		(pts
-			(xy 40.64 53.34) (xy 40.64 54.61)
+			(xy 222.25 76.2) (xy 222.25 78.74)
 		)
 		(stroke
@@
 	(wire
 		(pts
+			(xy 218.44 83.82) (xy 231.14 83.82)
+		)
+		(stroke
+			(width 0)
+			(type default)
+		)
+	)
+	(wire
+		(pts
 			(xy 25.4 44.45) (xy 27.94 44.45)
 		)
@@
 	(wire
 		(pts
-			(xy 31.75 146.05) (xy 41.91 146.05)
+			(xy 215.9 86.36) (xy 218.44 86.36)
+		)
+		(stroke
+			(width 0)
+			(type default)
+		)
+	)
+	(wire
+		(pts
+			(xy 30.48 146.05) (xy 41.91 146.05)
 		)
 		(stroke
@@
 	(wire
 		(pts
+			(xy 220.98 86.36) (xy 220.98 91.44)
+		)
+		(stroke
+			(width 0)
+			(type default)
+		)
+	)
+	(wire
+		(pts
 			(xy 76.2 53.34) (xy 76.2 55.88)
 		)
@@
 		)
 	)
-	(global_label "pwmgauche"
+	(global_label "pwmdroite"
 		(shape input)
-		(at 33.02 143.51 180)
+		(at 30.48 143.51 180)
 		(fields_autoplaced yes)
 		(effects
@@
 		)
 		(property "Intersheetrefs" "${INTERSHEET_REFS}"
-			(at 19.0888 143.51 0)
+			(at 17.8187 143.51 0)
 			(effects
 				(font
@@
 	(global_label "T2 sortie"
 		(shape input)
-		(at 215.9 85.09 180)
+		(at 215.9 86.36 180)
 		(fields_autoplaced yes)
 		(effects
@@
 		)
 		(property "Intersheetrefs" "${INTERSHEET_REFS}"
-			(at 204.3877 85.09 0)
+			(at 204.3877 86.36 0)
 			(effects
 				(font
@@
 	(global_label "T3 sortie"
 		(shape input)
-		(at 215.9 91.44 180)
+		(at 215.9 81.28 180)
 		(fields_autoplaced yes)
 		(effects
@@
 		)
 		(property "Intersheetrefs" "${INTERSHEET_REFS}"
-			(at 204.3877 91.44 0)
+			(at 204.3877 81.28 0)
 			(effects
 				(font
@@
 	(global_label "T1 sortie"
 		(shape input)
-		(at 215.9 78.74 180)
+		(at 215.9 91.44 180)
 		(fields_autoplaced yes)
 		(effects
@@
 		)
 		(property "Intersheetrefs" "${INTERSHEET_REFS}"
-			(at 204.3877 78.74 0)
+			(at 204.3877 91.44 0)
 			(effects
 				(font
@@
 	(global_label "T4 sortie"
 		(shape input)
-		(at 215.9 97.79 180)
+		(at 215.9 76.2 180)
 		(fields_autoplaced yes)
 		(effects
@@
 		)
 		(property "Intersheetrefs" "${INTERSHEET_REFS}"
-			(at 204.3877 97.79 0)
+			(at 204.3877 76.2 0)
 			(effects
 				(font
@@
 		)
 	)
-	(global_label "pwmdroite"
+	(global_label "pwmgauche"
 		(shape input)
-		(at 31.75 146.05 180)
+		(at 30.48 146.05 180)
 		(fields_autoplaced yes)
 		(effects
@@
 		)
 		(property "Intersheetrefs" "${INTERSHEET_REFS}"
-			(at 19.0887 146.05 0)
+			(at 16.5488 146.05 0)
 			(effects
 				(font
@@
 			)
 		)
-		(property "Footprint" "ampli op:LMC6482"
+		(property "Footprint" "ampli op:LMC6482_SMT"
 			(at 168.91 41.91 0)
 			(effects
@@
 			)
 		)
-		(property "Footprint" "ampli op:LMC6482"
+		(property "Footprint" "ampli op:LMC6482_SMT"
 			(at 86.36 99.06 0)
 			(effects
@@
 			)
 		)
-		(property "Footprint" "ampli op:LMC6482"
+		(property "Footprint" "ampli op:LMC6482_SMT"
 			(at 134.62 39.37 0)
 			(effects
@@
 			)
 		)
-		(property "Footprint" "ampli op:LMC6482"
+		(property "Footprint" "ampli op:LMC6482_SMT"
 			(at 168.91 95.25 0)
 			(effects
@@
 			)
 		)
-		(property "Footprint" "ampli op:LMC6482"
+		(property "Footprint" "ampli op:LMC6482_SMT"
 			(at 86.36 44.45 0)
 			(effects
@@
 		(on_board yes)
 		(dnp no)
-		(fields_autoplaced yes)
 		(property "Reference" "#PWR033"
 			(at 36.83 166.37 0)
@@
 			)
 		)
-		(property "Value" "+5V"
-			(at 29.21 166.3699 90)
+		(property "Value" "+5V (Ali seulement)"
+			(at 31.496 168.148 90)
 			(effects
 				(font
 					(size 1.27 1.27)
 				)
-				(justify left)
 			)
 		)
@@
 			)
 		)
-		(property "Footprint" "ampli op:LMC6482"
+		(property "Footprint" "ampli op:LMC6482_SMT"
 			(at 52.07 41.91 0)
 			(effects
@@
 			)
 		)
-		(property "Footprint" "ampli op:LMC6482"
+		(property "Footprint" "ampli op:LMC6482_SMT"
 			(at 52.07 96.52 0)
 			(effects
@@
 			)
 		)
-		(property "Footprint" "ampli op:LMC6482"
+		(property "Footprint" "ampli op:LMC6482_SMT"
 			(at 134.62 92.71 0)
 			(effects
@@
 		(on_board yes)
 		(dnp no)
-		(fields_autoplaced yes)
 		(property "Reference" "#PWR013"
 			(at 35.56 151.13 0)
@@
 			)
 		)
-		(property "Value" "+5V"
-			(at 27.94 151.1299 90)
+		(property "Value" "+5V (Ali seulement)"
+			(at 28.956 152.654 90)
 			(effects
 				(font
 					(size 1.27 1.27)
 				)
-				(justify left)
 			)
 		)

Commit message: PCB V2 - Envoyé à Martin
Parts:
- removed J2: Screw_Terminal_01x02, Connector_JST:JST_PH_B2B-PH-K_1x02_P2.00mm_Vertical, symbol Connector:Screw_Terminal_01x02
- added J2: Screw_Terminal_01x03, Connector_JST:JST_XH_B3B-XH-A_1x03_P2.50mm_Vertical, symbol Connector:Screw_Terminal_01x03
- J1: footprint Connector_JST:JST_PH_B4B-PH-K_1x04_P2.00mm_Vertical -> Connector_JST:JST_XH_B4B-XH-A_1x04_P2.50mm_Vertical
Connections:
- net +5V (Ali seulement): now also J2.2 (Pin_2)
- net GND: now also J2.1 (Pin_1)
Changed lines of the file:
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@@
 	)
 	(symbol
-		(lib_id "Connector:Screw_Terminal_01x02")
-		(at 46.99 163.83 0)
-		(unit 1)
-		(exclude_from_sim no)
-		(in_bom yes)
-		(on_board yes)
-		(dnp no)
-		(fields_autoplaced yes)
-		(property "Reference" "J2"
-			(at 49.53 163.8299 0)
-			(effects
-				(font
-					(size 1.27 1.27)
-				)
-				(justify left)
-			)
-		)
-		(property "Value" "Screw_Terminal_01x02"
-			(at 49.53 166.3699 0)
-			(effects
-				(font
-					(size 1.27 1.27)
-				)
-				(justify left)
-			)
-		)
-		(property "Footprint" "Connector_JST:JST_PH_B2B-PH-K_1x02_P2.00mm_Vertical"
-			(at 46.99 163.83 0)
-			(effects
-				(font
-					(size 1.27 1.27)
-				)
-				(hide yes)
-			)
-		)
-		(property "Datasheet" "~"
-			(at 46.99 163.83 0)
-			(effects
-				(font
-					(size 1.27 1.27)
-				)
-				(hide yes)
-			)
-		)
-		(property "Description" "Generic screw terminal, single row, 01x02, script generated (kicad-library-utils/schlib/autogen/connector/)"
-			(at 46.99 163.83 0)
-			(effects
-				(font
-					(size 1.27 1.27)
-				)
-				(hide yes)
-			)
-		)
-		(pin "1"
-		)
-		(pin "2"
-		)
-		(instances
-			(project ""
-				(path "/08655c7e-db3e-4a36-827c-446c5903f8cb"
-					(reference "J2")
-					(unit 1)
-				)
-			)
-		)
-	)
-	(symbol
 		(lib_id "Amplifier_Operational:LMC6482")
 		(at 134.62 39.37 0)
@@
 			)
 		)
-		(property "Footprint" "Connector_JST:JST_PH_B4B-PH-K_1x04_P2.00mm_Vertical"
+		(property "Footprint" "Connector_JST:JST_XH_B4B-XH-A_1x04_P2.50mm_Vertical"
 			(at 46.99 146.05 0)
 			(effects
@@
 					(unit 1)
 				)
+			)
+		)
+	)
+	(symbol
+		(lib_id "Connector:Screw_Terminal_01x03")
+		(at 46.99 166.37 0)
+		(unit 1)
+		(exclude_from_sim no)
+		(in_bom yes)
+		(on_board yes)
+		(dnp no)
+		(fields_autoplaced yes)
+		(property "Reference" "J2"
+			(at 49.53 165.0999 0)
+			(effects
+				(font
+					(size 1.27 1.27)
+				)
+				(justify left)
+			)
+		)
+		(property "Value" "Screw_Terminal_01x03"
+			(at 49.53 167.6399 0)
+			(effects
+				(font
+					(size 1.27 1.27)
+				)
+				(justify left)
+			)
+		)
+		(property "Footprint" "Connector_JST:JST_XH_B3B-XH-A_1x03_P2.50mm_Vertical"
+			(at 46.99 166.37 0)
+			(effects
+				(font
+					(size 1.27 1.27)
+				)
+				(hide yes)
+			)
+		)
+		(property "Datasheet" "~"
+			(at 46.99 166.37 0)
+			(effects
+				(font
+					(size 1.27 1.27)
+				)
+				(hide yes)
+			)
+		)
+		(property "Description" "Generic screw terminal, single row, 01x03, script generated (kicad-library-utils/schlib/autogen/connector/)"
+			(at 46.99 166.37 0)
+			(effects
+				(font
+					(size 1.27 1.27)
+				)
+				(hide yes)
+			)
+		)
+		(pin "3"
+		)
+		(pin "2"
+		)
+		(pin "1"
+		)
+		(instances
+			(project ""
+				(path "/08655c7e-db3e-4a36-827c-446c5903f8cb"
+					(reference "J2")
+					(unit 1)
+				)
