File: code arduino et fichiers kicad/kicad/pcb.kicad_pcb (KiCad board)
At the start: 2 copper layers, 53.5 x 80 mm, 46 parts, among them J1 Screw_Terminal_01x04, J2 Screw_Terminal_01x02, U1 LMC6482, U2 LMC6482, U3 LMC6482, U4 LMC6482

Commit message: PCB V2 - Envoyé à Martin
Parts:
- J1: footprint Connector_JST:JST_PH_B4B-PH-K_1x04_P2.00mm_Vertical -> Connector_JST:JST_XH_B4B-XH-A_1x04_P2.50mm_Vertical
- J2: value Screw_Terminal_01x02 -> Screw_Terminal_01x03; footprint Connector_JST:JST_PH_B2B-PH-K_1x02_P2.00mm_Vertical -> Connector_JST:JST_XH_B3B-XH-A_1x03_P2.50mm_Vertical
- moved R18 3.93 mm to (108.5, 52.7)
- moved D4 2.63 mm to (113.7, 53.9)
- moved J2 1.33 mm to (97.6, 49.2)
- moved J1 0.74 mm to (82.3, 49.2)
Routing:
- net GND: track 63.0 -> 61.7 mm
- net Net-(D4-A): track 7.20 -> 6.11 mm
- net pwmgauche: track 68.8 -> 69.8 mm
- net +5V (Ali seulement): track 13.0 -> 13.7 mm
- net pwmdroite: track 38.6 -> 39.3 mm
