File: pcb et ancienne identification/kicad/pcb.kicad_sch (KiCad schematic)
At the start: 46 parts, among them J1 MTA_02, J2 MTA_04, U1 LMC6482IMX_NOPB, U2 LMC6482IMX_NOPB, U3 LMC6482IMX_NOPB, U4 LMC6482IMX_NOPB

Commit message: impression schéma électrique pour éval prototype
Other:
- note added: "Arduino Mega 2560"
- note added: "Circuit d'alimentation"
- note added: "Circuit de conditionnement"
- note removed: "circuit d'alimentation"
- note removed: "circuit de conditionnement"
- title: (none) -> Circuit électrique prototype plaque thermique
- moved on the sheet: C1, C2, C3, C4, D1, J1, J2, R1, R10, R11, R12, R13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
